Commit message: update

File: blimp_description/urdf/description_controller.xacro (robot description, xacro)
@@ -45,5 +45,5 @@
 		link_name="bot_rud_motor_link"
 		direction="cw"
-		motor_constant="${motor_constant}"
+		motor_constant="${bot_motor_constant}"
 		moment_constant="${moment_constant}"
 		time_constant_up="${time_constant_up}"

File: blimp_description/urdf/description_property.xacro (robot description, xacro)
@@ -66,5 +66,6 @@
 	<xacro:property name="rotor_velocity_slowdown_sim" value="1" />
 	<xacro:property name="rotor_offset_top" value="0.05" /> <!-- [m] -->
-	<xacro:property name="motor_constant" value="3.71178707e-03" /> <!-- [kg m/s^2] -->
+	<xacro:property name="motor_constant" value="3.71178707e-03" /> <!-- [kg m/s^2], default: 3.71178707e-03 -->
+	<xacro:property name="bot_motor_constant" value="3.71178707e-03" /> <!-- [kg m/s^2], default: 3.71178707e-03 -->
 	<xacro:property name="moment_constant" value="0.016" /> <!-- [m] -->
 	<!--<xacro:property name="time_constant_up" value="0.0125" /> --><!-- [s] -->
